File: FiberLink.brd (EAGLE design)
At the start: 50 x 25 mm, 76 parts, among them X1 629105136821

Commit message: PDF Layout added
Parts:
- added DRILEGEND: (no value), drilegend:DRILEGEND

Commit message: Configuration documentation added
Parts:
- SJ10: value (none) -> 10
- SJ11: value (none) -> 11
- SJ12: value (none) -> 12
- SJ13: value (none) -> 13
- SJ14: value (none) -> 14
- SJ15: value (none) -> 15
- SJ17: value SJ-TRI -> 17
- SJ2: value (none) -> 2
- SJ3: value (none) -> 3
- SJ4: value (none) -> 4
- SJ5: value (none) -> 5
- SJ6: value (none) -> 6
- SJ7: value (none) -> 7
- SJ8: value (none) -> 8
- SJ9: value (none) -> 9
Other:
- board text added: "SJ2 FIBER RX TO RS232 SJ3 FIBER RX TO USB SJ4 RS232 RX TO FIBER SJ5 USB RX TO FIBER SJ6 USB RX TO RS232 SJ7 RS232 RX TO USB SJ8 RS485 RX TO FIBER SJ9 FIBER RX TO RS485 SJ10 RS485 RX TO USB SJ11 USB RX TO RS485 SJ12 RS232 RX TO RS485 SJ13 RS485 RX TO RS232 SJ14 CARRIER SENSE TO RX485 TXEN SJ15 USB TXEN TO RS485 TXEN SJ17 FTDI POWER SELECT (UP=BUS, DOWN=SELF)"
- board text added: "USB <-> RS232 SJ6, SJ7 USB <-> RS485 SJ10, SJ11, SJ15 USB <-> FIBER SJ3, SJ5 RS232 <-> RS485 SJ12, SJ13, SJ14 RS232 <-> FIBER SJ2, SJ4 FIBER <-> RS485 SJ8, SJ9, SJ14"
