File: FiberLink.sch (EAGLE design)
At the start: 76 parts, among them X1 629105136821

Commit message: Configuration documentation added
Parts:
- SJ10: value (none) -> 10
- SJ11: value (none) -> 11
- SJ12: value (none) -> 12
- SJ13: value (none) -> 13
- SJ14: value (none) -> 14
- SJ15: value (none) -> 15
- SJ17: value SJ-TRI -> 17
- SJ2: value (none) -> 2
- SJ3: value (none) -> 3
- SJ4: value (none) -> 4
- SJ5: value (none) -> 5
- SJ6: value (none) -> 6
- SJ7: value (none) -> 7
- SJ8: value (none) -> 8
- SJ9: value (none) -> 9
Other:
- note added: "SJ2 FIBER RX TO RS232 SJ3 FIBER RX TO USB SJ4 RS232 RX TO FIBER SJ5 USB RX TO FIBER SJ6 USB RX TO RS232 SJ7 RS232 RX TO USB SJ8 RS485 RX TO FIBER SJ9 FIBER RX TO RS485 SJ10 RS485 RX TO USB SJ11 USB RX TO RS485 SJ12 RS232 RX TO RS485 SJ13 RS485 RX TO RS232 SJ14 CARRIER SENSE TO RX485 TXEN SJ15 USB TXEN TO RS485 TXEN SJ17 FTDI POWER SELECT"
- note added: "USB <-> RS232 SJ6, SJ7 USB <-> RS485 SJ10, SJ11, SJ15 USB <-> FIBER SJ3, SJ5 RS232 <-> RS485 SJ12, SJ13, SJ14 RS232 <-> FIBER SJ2, SJ4 FIBER <-> RS485 SJ8, SJ9, SJ14"
- moved on the sheet: R28, R9
Changed lines of the file:
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@@
 <part name="GND18" library="supply1" deviceset="GND" device=""/>
 <part name="V2" library="diode" deviceset="DIODE-" device="SOD323-R"/>
-<part name="SJ2" library="OMAT_IC" deviceset="SJ" device=""/>
-<part name="SJ3" library="OMAT_IC" deviceset="SJ" device=""/>
-<part name="SJ4" library="OMAT_IC" deviceset="SJ" device=""/>
-<part name="SJ5" library="OMAT_IC" deviceset="SJ" device=""/>
-<part name="SJ6" library="OMAT_IC" deviceset="SJ" device=""/>
-<part name="SJ7" library="OMAT_IC" deviceset="SJ" device=""/>
-<part name="SJ8" library="OMAT_IC" deviceset="SJ" device=""/>
-<part name="SJ9" library="OMAT_IC" deviceset="SJ" device=""/>
-<part name="SJ10" library="OMAT_IC" deviceset="SJ" device=""/>
-<part name="SJ11" library="OMAT_IC" deviceset="SJ" device=""/>
-<part name="SJ12" library="OMAT_IC" deviceset="SJ" device=""/>
-<part name="SJ13" library="OMAT_IC" deviceset="SJ" device=""/>
-<part name="SJ14" library="OMAT_IC" deviceset="SJ" device=""/>
-<part name="SJ15" library="OMAT_IC" deviceset="SJ" device=""/>
+<part name="SJ2" library="OMAT_IC" deviceset="SJ" device="" value="2"/>
+<part name="SJ3" library="OMAT_IC" deviceset="SJ" device="" value="3"/>
+<part name="SJ4" library="OMAT_IC" deviceset="SJ" device="" value="4"/>
+<part name="SJ5" library="OMAT_IC" deviceset="SJ" device="" value="5"/>
+<part name="SJ6" library="OMAT_IC" deviceset="SJ" device="" value="6"/>
+<part name="SJ7" library="OMAT_IC" deviceset="SJ" device="" value="7"/>
+<part name="SJ8" library="OMAT_IC" deviceset="SJ" device="" value="8"/>
+<part name="SJ9" library="OMAT_IC" deviceset="SJ" device="" value="9"/>
+<part name="SJ10" library="OMAT_IC" deviceset="SJ" device="" value="10"/>
+<part name="SJ11" library="OMAT_IC" deviceset="SJ" device="" value="11"/>
+<part name="SJ12" library="OMAT_IC" deviceset="SJ" device="" value="12"/>
+<part name="SJ13" library="OMAT_IC" deviceset="SJ" device="" value="13"/>
+<part name="SJ14" library="OMAT_IC" deviceset="SJ" device="" value="14"/>
+<part name="SJ15" library="OMAT_IC" deviceset="SJ" device="" value="15"/>
 <part name="V1" library="OMAT_IC" deviceset="IFD91" device=""/>
 <part name="H1" library="OMAT_IC" deviceset="IFE91A" device=""/>
@@
 <part name="P+16" library="supply1" deviceset="+5V" device=""/>
 <part name="GND24" library="supply1" deviceset="GND" device=""/>
-<part name="SJ17" library="OMAT_IC" deviceset="SJ-TRI" device=""/>
+<part name="SJ17" library="OMAT_IC" deviceset="SJ-TRI" device="" value="17"/>
 </parts>
 <sheets>
 <sheet>
 <plain>
+<text x="144.78" y="-5.08" size="1.778" layer="91">SJ2 FIBER RX TO RS232
+SJ3 FIBER RX TO USB
+SJ4 RS232 RX TO FIBER
+SJ5 USB RX TO FIBER
+SJ6 USB RX TO RS232
+SJ7 RS232 RX TO USB
+SJ8 RS485 RX TO FIBER
+SJ9 FIBER RX TO RS485
+SJ10 RS485 RX TO USB
+SJ11 USB RX TO RS485
+SJ12 RS232 RX TO RS485
+SJ13 RS485 RX TO RS232
+SJ14 CARRIER SENSE TO RX485 TXEN
+SJ15 USB TXEN TO RS485 TXEN
+SJ17 FTDI POWER SELECT</text>
+<text x="200.66" y="-10.16" size="1.778" layer="91">USB &lt;-&gt; RS232
+SJ6, SJ7
+USB &lt;-&gt; RS485
+SJ10, SJ11, SJ15
+USB &lt;-&gt; FIBER
+SJ3, SJ5
+RS232 &lt;-&gt; RS485
+SJ12, SJ13, SJ14
+RS232 &lt;-&gt; FIBER
+SJ2, SJ4
+FIBER &lt;-&gt; RS485
+SJ8, SJ9, SJ14</text>
 </plain>
 <instances>
@@
 </instance>
 <instance part="R8" gate="G$1" x="157.48" y="111.76" rot="MR270"/>
-<instance part="R9" gate="G$1" x="165.1" y="96.52" rot="R270"/>
+<instance part="R9" gate="G$1" x="162.56" y="96.52" rot="R270"/>
 <instance part="X2" gate="G$1" x="398.78" y="50.8" rot="MR0"/>
 <instance part="GND8" gate="1" x="383.54" y="35.56" rot="MR0"/>
@@
 <instance part="GND17" gate="1" x="378.46" y="91.44"/>
 <instance part="X3" gate="1" x="401.32" y="121.92" rot="R180"/>
-<instance part="R28" gate="G$1" x="165.1" y="124.46" rot="R270"/>
+<instance part="R28" gate="G$1" x="162.56" y="124.46" rot="R270"/>
 <instance part="R29" gate="G$1" x="157.48" y="88.9" rot="MR270"/>
 <instance part="C16" gate="G$1" x="208.28" y="99.06" rot="R180"/>
@@
 <instance part="GND24" gate="1" x="373.38" y="-55.88"/>
 <instance part="SJ17" gate="G$1" x="248.92" y="-38.1" smashed="yes">
-<attribute name="NAME" x="246.38" y="-46.99" size="1.778" layer="95"/>
-<attribute name="VALUE" x="246.38" y="-43.18" size="1.778" layer="96"/>
+<attribute name="NAME" x="246.38" y="-44.45" size="1.778" layer="95"/>
+<attribute name="VALUE" x="246.38" y="-43.18" size="1.778" layer="96" display="off"/>
 </instance>
 </instances>
@@
 <pinref part="R9" gate="G$1" pin="2"/>
 <wire x1="172.72" y1="91.44" x2="172.72" y2="99.06" width="0.1524" layer="91"/>
-<wire x1="172.72" y1="91.44" x2="165.1" y2="91.44" width="0.1524" layer="91"/>
+<wire x1="172.72" y1="91.44" x2="162.56" y2="91.44" width="0.1524" layer="91"/>
 <junction x="172.72" y="91.44"/>
 </segment>
@@
 <pinref part="R28" gate="G$1" pin="1"/>
 <wire x1="172.72" y1="132.08" x2="172.72" y2="134.62" width="0.1524" layer="91"/>
-<wire x1="165.1" y1="129.54" x2="165.1" y2="132.08" width="0.1524" layer="91"/>
-<wire x1="165.1" y1="132.08" x2="172.72" y2="132.08" width="0.1524" layer="91"/>
+<wire x1="162.56" y1="129.54" x2="162.56" y2="132.08" width="0.1524" layer="91"/>
+<wire x1="162.56" y1="132.08" x2="172.72" y2="132.08" width="0.1524" layer="91"/>
 <junction x="172.72" y="132.08"/>
 </segment>
@@
 <segment>
 <pinref part="R9" gate="G$1" pin="1"/>
-<wire x1="165.1" y1="101.6" x2="165.1" y2="109.22" width="0.1524" layer="91"/>
+<wire x1="162.56" y1="101.6" x2="162.56" y2="109.22" width="0.1524" layer="91"/>
+<pinref part="R28" gate="G$1" pin="2"/>
+<wire x1="162.56" y1="109.22" x2="162.56" y2="119.38" width="0.1524" layer="91"/>
 <pinref part="N1" gate="A" pin="+IN"/>
-<pinref part="R28" gate="G$1" pin="2"/>
-<wire x1="165.1" y1="109.22" x2="165.1" y2="119.38" width="0.1524" layer="91"/>
-<junction x="165.1" y="109.22"/>
+<wire x1="165.1" y1="109.22" x2="162.56" y2="109.22" width="0.1524" layer="91"/>
+<junction x="162.56" y="109.22"/>
 </segment>
 </net>
@@
 </schematic>
 </drawing>
+<compatibility>
+<note version="6.3" minversion="6.2.2" severity="warning">
+Since Version 6.2.2 text objects can contain more than one line,
+which will not be processed correctly with this version.
+</note>
+</compatibility>
 </eagle>
